File: pcb/Omi-Glass-DevKit.kicad_sch (KiCad schematic)
At the start: 33 parts, among them J1 Conn_01x02, J2 Conn_01x02, J3 Conn_01x02, J5 0.5mm FFC 24, SW1 SW_Push, U1 NCP163AFCS280T2G, U2 NCP163AFCT180T2G

Commit message: bump to R0.2 V3
Parts:
- removed JP1: Jumper_2_Open, symbol Jumper:Jumper_2_Open
Connections:
- net VBAT1 is gone; now on net LOAD: J1.2 (Pin_2)
Changed lines of the file:
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@@
+	)
+	(junction
+		(at 99.06 167.64)
+		(diameter 0)
+		(color 0 0 0 0)
+	)
+	(junction
+		(at 100.33 55.88)
+		(diameter 0)
+		(color 0 0 0 0)
+	)
+	(junction
+		(at 93.98 167.64)
+		(diameter 0)
+		(color 0 0 0 0)
+	)
+	(junction
+		(at 68.58 133.35)
+		(diameter 0)
+		(color 0 0 0 0)
+	)
+	(junction
+		(at 107.95 101.6)
+		(diameter 0)
+		(color 0 0 0 0)
 	)
 	(junction
@@
 	)
 	(junction
-		(at 99.06 167.64)
-		(diameter 0)
-		(color 0 0 0 0)
-	)
-	(junction
-		(at 100.33 55.88)
-		(diameter 0)
-		(color 0 0 0 0)
-	)
-	(junction
-		(at 93.98 167.64)
-		(diameter 0)
-		(color 0 0 0 0)
-	)
-	(junction
-		(at 246.38 63.5)
-		(diameter 0)
-		(color 0 0 0 0)
-	)
-	(junction
-		(at 68.58 133.35)
-		(diameter 0)
-		(color 0 0 0 0)
-	)
-	(junction
-		(at 256.54 63.5)
+		(at 113.03 101.6)
 		(diameter 0)
 		(color 0 0 0 0)
@@
 	)
 	(junction
-		(at 107.95 101.6)
-		(diameter 0)
-		(color 0 0 0 0)
-	)
-	(junction
-		(at 113.03 101.6)
-		(diameter 0)
-		(color 0 0 0 0)
-	)
-	(junction
 		(at 265.43 63.5)
 		(diameter 0)
@@
 	(wire
 		(pts
-			(xy 246.38 63.5) (xy 240.03 63.5)
-		)
-		(stroke
-			(width 0)
-			(type default)
-		)
-	)
-	(wire
-		(pts
 			(xy 201.93 114.3) (xy 201.93 116.84)
 		)
@@
 	(wire
 		(pts
-			(xy 262.89 63.5) (xy 256.54 63.5)
-		)
-		(stroke
-			(width 0)
-			(type default)
-		)
-	)
-	(wire
-		(pts
 			(xy 100.33 60.96) (xy 100.33 55.88)
 		)
@@
 	(wire
 		(pts
+			(xy 240.03 63.5) (xy 262.89 63.5)
+		)
+		(stroke
+			(width 0)
+			(type default)
+		)
+	)
+	(wire
+		(pts
 			(xy 220.98 36.83) (xy 220.98 43.18)
 		)
@@
 		(pts
 			(xy 227.33 140.97) (xy 227.457 140.97)
-		)
-		(stroke
-			(width 0)
-			(type default)
-		)
-	)
-	(wire
-		(pts
-			(xy 256.54 63.5) (xy 255.27 63.5)
-		)
-		(stroke
-			(width 0)
-			(type default)
-		)
-	)
-	(wire
-		(pts
-			(xy 247.65 63.5) (xy 246.38 63.5)
 		)
 		(stroke
@@
 					(unit 1)
 				)
-			)
-		)
-	)
-	(symbol
-		(lib_id "Jumper:Jumper_2_Open")
-		(at 251.46 63.5 0)
-		(unit 1)
-		(exclude_from_sim no)
-		(in_bom yes)
-		(on_board yes)
-		(dnp no)
-		(fields_autoplaced yes)
-		(property "Reference" "JP1"
-			(at 251.46 57.15 0)
-			(effects
-				(font
-					(size 1.27 1.27)
-				)
-			)
-		)
-		(property "Value" "Jumper_2_Open"
-			(at 251.46 59.69 0)
-			(effects
-				(font
-					(size 1.27 1.27)
-				)
-			)
-		)
-		(property "Footprint" ""
-			(at 251.46 63.5 0)
-			(effects
-				(font
-					(size 1.27 1.27)
-				)
-				(hide yes)
-			)
-		)
-		(property "Datasheet" "~"
-			(at 251.46 63.5 0)
-			(effects
-				(font
-					(size 1.27 1.27)
-				)
-				(hide yes)
-			)
-		)
-		(property "Description" "Jumper, 2-pole, open"
-			(at 251.46 63.5 0)
-			(effects
-				(font
-					(size 1.27 1.27)
-				)
-				(hide yes)
-			)
-		)
-		(pin "1"
-		)
-		(pin "2"
-		)
-		(instances
-			(project ""
-				(path "/635eb50f-488a-4d6f-8ee4-97bdde581e20"
-					(reference "JP1")
-					(unit 1)
-				)
